File: hardware/board.brd (EAGLE design)
At the start: 63.8 x 43.7 mm, 82 parts, among them J6 51281-0594, Q2 2.5A/30V/105mΩ, Q3 2.5A/30V/105mΩ, Q4 2.5A/30V/105mΩ, Q5 5.8A/30V/35mΩ, Q6 2.5A/30V/105mΩ, U1 DRV8837DSGR, U3 MB85RC256VPF-G-JNERE2, U4 MAX9934TAUA, U5 BQ25570RGRR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

Commit message: Add files
Parts:
- C21: value 2.2uF -> 0.6F
- L2: value 3.3µH/±20%/450mA -> 10uH
- R10, R7: value 1K -> 1
- R25: value 820k -> 820K
- R26: value 2.0M -> 2M
Connections:
- removed net N$5: D4.1, Q4.2
- net 3.3V: no longer R5.2, R9.2
- net A5: now also D4.1, Q4.2
- net N$12: now also R5.2, R9.2
Routing:
- net A5: track 24.0 -> 67.8 mm, vias 2 -> 6
- net N$5: track 16.9 -> 0.00 mm
- net N$12: track 8.18 -> 18.1 mm
- net 3.3V: track 138.1 -> 130.8 mm, vias 9 -> 8
- net IBATT: track 47.3 -> 49.3 mm
- net VINM: track 42.8 -> 44.0 mm
