File: hardware/board.sch (EAGLE design)
At the start: 82 parts, among them J6 51281-0594, Q1 MOSFET_PCH-DMG2307L, Q2 2.5A/30V/105mΩ, Q3 2.5A/30V/105mΩ, Q4 2.5A/30V/105mΩ, Q5 5.8A/30V/35mΩ, Q6 2.5A/30V/105mΩ, U1 DRV8837DSGR, U3 MB85RC256VPF-G-JNERE2, U4 MAX9934TAUA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

Commit message: Add files
Parts:
- C21: value 2.2uF -> 0.6F
- L2: value 3.3µH/±20%/450mA -> 10uH
- R10, R7: value 1K -> 1
- R25: value 820k -> 820K
- R26: value 2.0M -> 2M
Connections:
- removed net N$5: D4.+, Q4.S
- net 3.3V: no longer R5.2, R9.2
- net A5: now also D4.+, Q4.S
- net N$12: now also R5.2, R9.2
Other:
- note added: "Don't use this"
Changed lines of the file:
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@@
 <part name="J6" library="51281-0594" deviceset="51281-0594" device=""/>
 <part name="JP2" library="SparkFun-Jumpers" library_urn="urn:adsk.eagle:library:528" deviceset="JUMPER-SMT_2_NO" device="_SILK" package3d_urn="urn:adsk.eagle:package:39279/1"/>
-<part name="C21" library="SparkFun-Capacitors" library_urn="urn:adsk.eagle:library:510" deviceset="2.2UF" device="-0805-25V-(+80/-20%)" package3d_urn="urn:adsk.eagle:package:37429/1" value="2.2uF"/>
+<part name="C21" library="SparkFun-Capacitors" library_urn="urn:adsk.eagle:library:510" deviceset="2.2UF" device="-0805-25V-(+80/-20%)" package3d_urn="urn:adsk.eagle:package:37429/1" value="0.6F"/>
 <part name="GND42" library="SparkFun-PowerSymbols" library_urn="urn:adsk.eagle:library:530" deviceset="GND" device=""/>
 <part name="U$2" library="SOT65P280X145-8N" deviceset="AD5273" device=""/>
@@
 <part name="R24" library="SparkFun-Resistors" library_urn="urn:adsk.eagle:library:532" deviceset="1KOHM" device="-0603-1/10W-1%" package3d_urn="urn:adsk.eagle:package:39650/1" value="1k"/>
 <part name="J7" library="SparkFun-Connectors" deviceset="CONN_02" device="" package3d_urn="urn:adsk.eagle:package:38039/1"/>
-<part name="R7" library="SparkFun-Resistors" library_urn="urn:adsk.eagle:library:532" deviceset="0.05OHM" device="-0603-1/5W-1%" package3d_urn="urn:adsk.eagle:package:39650/1" value="1K"/>
+<part name="R7" library="SparkFun-Resistors" library_urn="urn:adsk.eagle:library:532" deviceset="0.05OHM" device="-0603-1/5W-1%" package3d_urn="urn:adsk.eagle:package:39650/1" value="1"/>
 <part name="D4" library="Comchip - CDBHD140L-G" deviceset="COMCHIP_CDBHD140L-G" device="COMCHIP_CDBHD140L-G_0_0"/>
 <part name="Q4" library="SparkFun-DiscreteSemi" library_urn="urn:adsk.eagle:library:514" deviceset="MOSFET_PCH" device="-DMG2307L" package3d_urn="urn:adsk.eagle:package:38446/1" value="2.5A/30V/105mΩ"/>
@@
 <part name="SUPPLY6" library="SparkFun-PowerSymbols" library_urn="urn:adsk.eagle:library:530" deviceset="3.3V" device=""/>
 <part name="Q2" library="SparkFun-DiscreteSemi" library_urn="urn:adsk.eagle:library:514" deviceset="MOSFET_PCH" device="-DMG2307L" package3d_urn="urn:adsk.eagle:package:38446/1" value="2.5A/30V/105mΩ"/>
-<part name="R25" library="SparkFun-Resistors" library_urn="urn:adsk.eagle:library:532" deviceset="820KOHM" device="-0603-1/10W-1%" package3d_urn="urn:adsk.eagle:package:39650/1" value="820k"/>
-<part name="R26" library="SparkFun-Resistors" library_urn="urn:adsk.eagle:library:532" deviceset="2MOHMS" device="-0603-1/10W-1%" package3d_urn="urn:adsk.eagle:package:39650/1" value="2.0M"/>
+<part name="R25" library="SparkFun-Resistors" library_urn="urn:adsk.eagle:library:532" deviceset="820KOHM" device="-0603-1/10W-1%" package3d_urn="urn:adsk.eagle:package:39650/1" value="820K"/>
+<part name="R26" library="SparkFun-Resistors" library_urn="urn:adsk.eagle:library:532" deviceset="2MOHMS" device="-0603-1/10W-1%" package3d_urn="urn:adsk.eagle:package:39650/1" value="2M"/>
 <part name="SUPPLY22" library="SparkFun-PowerSymbols" library_urn="urn:adsk.eagle:library:530" deviceset="VIN" device=""/>
 <part name="GND23" library="SparkFun-PowerSymbols" library_urn="urn:adsk.eagle:library:530" deviceset="GND" device=""/>
@@
 <part name="R5" library="SparkFun-Resistors" library_urn="urn:adsk.eagle:library:532" deviceset="10KOHM" device="-0603-1/10W-1%" package3d_urn="urn:adsk.eagle:package:39650/1" value="10k"/>
 <part name="R9" library="SparkFun-Resistors" library_urn="urn:adsk.eagle:library:532" deviceset="10KOHM" device="-0603-1/10W-1%" package3d_urn="urn:adsk.eagle:package:39650/1" value="10k"/>
-<part name="SUPPLY15" library="SparkFun-PowerSymbols" library_urn="urn:adsk.eagle:library:530" deviceset="3.3V" device=""/>
 <part name="Q5" library="SparkFun-DiscreteSemi" library_urn="urn:adsk.eagle:library:514" deviceset="MOSFET-NCH" device="-AO3404A" package3d_urn="urn:adsk.eagle:package:38446/1" value="5.8A/30V/35mΩ"/>
 <part name="GND17" library="SparkFun-PowerSymbols" library_urn="urn:adsk.eagle:library:530" deviceset="GND" device=""/>
@@
 <part name="SUPPLY5" library="SparkFun-PowerSymbols" library_urn="urn:adsk.eagle:library:530" deviceset="3.3V" device=""/>
 <part name="J5" library="SparkFun-Connectors" deviceset="CONN_02" device="" package3d_urn="urn:adsk.eagle:package:38039/1"/>
-<part name="R10" library="SparkFun-Resistors" library_urn="urn:adsk.eagle:library:532" deviceset="1OHM" device="-0603-1/10W-1%" package3d_urn="urn:adsk.eagle:package:39650/1" value="1K"/>
+<part name="R10" library="SparkFun-Resistors" library_urn="urn:adsk.eagle:library:532" deviceset="1OHM" device="-0603-1/10W-1%" package3d_urn="urn:adsk.eagle:package:39650/1" value="1"/>
 <part name="U6" library="MAX9934TAUA" deviceset="MAX9934TAUA" device=""/>
 <part name="GND18" library="SparkFun-PowerSymbols" library_urn="urn:adsk.eagle:library:530" deviceset="GND" device=""/>
@@
 <part name="GND27" library="SparkFun-PowerSymbols" library_urn="urn:adsk.eagle:library:530" deviceset="GND" device=""/>
 <part name="GND31" library="SparkFun-PowerSymbols" library_urn="urn:adsk.eagle:library:530" deviceset="GND" device=""/>
-<part name="L2" library="SparkFun-Coils" library_urn="urn:adsk.eagle:library:512" deviceset="INDUCTOR" device="-0805-3.3UH" package3d_urn="urn:adsk.eagle:package:37579/1" value="3.3µH/±20%/450mA"/>
+<part name="L2" library="SparkFun-Coils" library_urn="urn:adsk.eagle:library:512" deviceset="INDUCTOR" device="-0805-3.3UH" package3d_urn="urn:adsk.eagle:package:37579/1" value="10uH"/>
 <part name="C14" library="SparkFun-Capacitors" library_urn="urn:adsk.eagle:library:510" deviceset="1.0UF" device="-0805-25V-(+80/-20%)" package3d_urn="urn:adsk.eagle:package:37429/1" value="4.7uF"/>
 <part name="C22" library="SparkFun-Capacitors" library_urn="urn:adsk.eagle:library:510" deviceset="0.1UF" device="-0603-25V-(+80/-20%)" package3d_urn="urn:adsk.eagle:package:37414/1" value="0.1uF"/>
@@
 <wire x1="-128.524" y1="123.698" x2="-91.44" y2="123.698" width="0.254" layer="94" style="longdash"/>
 <text x="-377.452" y="88.812" size="3.81" layer="94">NFC</text>
+<text x="-317.5" y="-20.32" size="1.778" layer="95">Don't use this</text>
+<text x="-317.5" y="-15.24" size="1.778" layer="95">Don't use this</text>
 </plain>
 <instances>
@@
 <instance part="C21" gate="G$1" x="-274.32" y="170.18" smashed="yes">
 <attribute name="NAME" x="-268.224" y="174.879" size="1.778" layer="95" font="vector" rot="R180"/>
+<attribute name="VALUE" x="-265.684" y="169.799" size="1.778" layer="96" font="vector" rot="R180"/>
 </instance>
 <instance part="GND42" gate="1" x="13.97" y="4.826" smashed="yes">
@@
 <attribute name="NAME" x="-55.88" y="87.884" size="1.778" layer="95" font="vector" align="bottom-center"/>
 <attribute name="VALUE" x="-60.96" y="89.916" size="1.778" layer="96" font="vector" align="top-center"/>
-</instance>
-<instance part="SUPPLY15" gate="G$1" x="-45.72" y="96.52" smashed="yes">
-<attribute name="VALUE" x="-45.72" y="99.314" size="1.778" layer="96" align="bottom-center"/>
 </instance>
 <instance part="Q5" gate="NMOS" x="-276.86" y="-63.5" smashed="yes">
@@
 </segment>
 <segment>
-<pinref part="R5" gate="G$1" pin="2"/>
-<wire x1="-55.88" y1="96.52" x2="-50.8" y2="96.52" width="0.1524" layer="91"/>
-<wire x1="-50.8" y1="96.52" x2="-50.8" y2="93.98" width="0.1524" layer="91"/>
-<pinref part="R9" gate="G$1" pin="2"/>
-<wire x1="-50.8" y1="93.98" x2="-50.8" y2="91.44" width="0.1524" layer="91"/>
-<wire x1="-50.8" y1="91.44" x2="-55.88" y2="91.44" width="0.1524" layer="91"/>
-<pinref part="SUPPLY15" gate="G$1" pin="3.3V"/>
-<wire x1="-45.72" y1="96.52" x2="-45.72" y2="93.98" width="0.1524" layer="91"/>
-<wire x1="-45.72" y1="93.98" x2="-50.8" y2="93.98" width="0.1524" layer="91"/>
-<junction x="-50.8" y="93.98"/>
-</segment>
-<segment>
 <pinref part="SUPPLY5" gate="G$1" pin="3.3V"/>
 <pinref part="Q6" gate="G$1" pin="S"/>
@@
 </segment>
 </net>
-<net name="N$5" class="0">
-<segment>
-<pinref part="D4" gate="G$0" pin="+"/>
-<wire x1="-312.42" y1="175.26" x2="-309.88" y2="175.26" width="0.1524" layer="91"/>
-<wire x1="-309.88" y1="195.58" x2="-309.88" y2="175.26" width="0.1524" layer="91"/>
-<pinref part="Q4" gate="G$1" pin="S"/>
-<wire x1="-297.18" y1="193.04" x2="-297.18" y2="195.58" width="0.1524" layer="91"/>
-<wire x1="-297.18" y1="195.58" x2="-309.88" y2="195.58" width="0.1524" layer="91"/>
-</segment>
-</net>
 <net name="RECEN" class="0">
 <segment>
@@
 <wire x1="-73.66" y1="78.74" x2="-73.66" y2="83.82" width="0.1524" layer="91"/>
 <junction x="-73.66" y="83.82"/>
+<wire x1="-73.66" y1="83.82" x2="-73.66" y2="86.36" width="0.1524" layer="91"/>
+<wire x1="-73.66" y1="86.36" x2="-45.72" y2="86.36" width="0.1524" layer="91"/>
+<pinref part="R5" gate="G$1" pin="2"/>
+<wire x1="-55.88" y1="96.52" x2="-50.8" y2="96.52" width="0.1524" layer="91"/>
+<wire x1="-50.8" y1="96.52" x2="-50.8" y2="93.98" width="0.1524" layer="91"/>
+<pinref part="R9" gate="G$1" pin="2"/>
+<wire x1="-50.8" y1="93.98" x2="-50.8" y2="91.44" width="0.1524" layer="91"/>
+<wire x1="-50.8" y1="91.44" x2="-55.88" y2="91.44" width="0.1524" layer="91"/>
+<wire x1="-45.72" y1="86.36" x2="-45.72" y2="93.98" width="0.1524" layer="91"/>
+<wire x1="-45.72" y1="93.98" x2="-50.8" y2="93.98" width="0.1524" layer="91"/>
+<junction x="-50.8" y="93.98"/>
 </segment>
 </net>
@@
 <label x="-287.02" y="-38.1" size="1.778" layer="95"/>
 </segment>
-</net>
+<segment>
+<pinref part="D4" gate="G$0" pin="+"/>
+<wire x1="-312.42" y1="175.26" x2="-309.88" y2="175.26" width="0.1524" layer="91"/>
+<wire x1="-309.88" y1="195.58" x2="-309.88" y2="175.26" width="0.1524" layer="91"/>
+<pinref part="Q4" gate="G$1" pin="S"/>
+<wire x1="-297.18" y1="193.04" x2="-297.18" y2="195.58" width="0.1524" layer="91"/>
+<wire x1="-297.18" y1="195.58" x2="-309.88" y2="195.58" width="0.1524" layer="91"/>
+<label x="-307.34" y="195.58" size="1.778" layer="95"/>
+</segment>
+</net>
